File: KiCAD/AnVCO/Antilog_NPNO.sch (KiCad schematic (older format))
At the start: 33 parts, among them J6 MSTR_OUT, J7 COURSE_SW, J8 MOD1, J9 MOD2, Q1 2SC1815, Q2 2SC1815, U1 TL072

Commit message: Before wiring
Parts:
- removed J8: MOD1, Connector_JST:JST_XH_B2B-XH-A_1x02_P2.50mm_Vertical, symbol Connector_Generic:Conn_01x02
- removed J9: MOD2, Connector_JST:JST_XH_B2B-XH-A_1x02_P2.50mm_Vertical, symbol Connector_Generic:Conn_01x02
- added J9: MOD, Connector_JST:JST_XH_B4B-XH-A_1x04_P2.50mm_Vertical, symbol Connector_Generic:Conn_01x04
- added JP2: TP_I_SINK, TestPoint:TestPoint_2Pads_Pitch2.54mm_Drill0.8mm, symbol Jumper:Jumper_2_Bridged
- added RV6: 50k/A, Potentiometer_THT:Potentiometer_Alps_RK097_Single_Horizontal, symbol Device:R_POT
- added TP2: TP_VREF, TestPoint:TestPoint_Pad_D1.0mm, symbol Connector:TestPoint
- RV1: footprint (none) -> Potentiometer_THT:Potentiometer_Bourns_3296W_Vertical
- TP1: value TP_ADJ -> TP_CV
- renumbered J6 to J7, J7 to J8
Connections:
- net GND: now also U1.3 (+), U1.5 (+), J9.2 (Pin_2), J9.4 (Pin_4), RV6.1; no longer U1.3 (+), U1.5 (+)
- net I_SINK: now also JP2.1 (A); no longer Q2.2 (C)
- net VREF: now also U1.2 (-), TP2.1; no longer U1.6 (-)
- net at RV5.3: now also J9.1 (Pin_1)
- net at R20.1, RV4.2, RV4.3: now also U1.7; no longer U1.1
- net at R10.2, R15.1, R19.1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: now also TP1.1, U1.6 (-); no longer U1.2 (-)
- net at R10.1, RV3.2: no longer TP1.1
- net at C6.1, R21.2: now also U1.1; no longer U1.7
- net at R22.2: now also RV6.2
- new net: JP2.2 (B), Q2.2 (C)
- new net: J9.3 (Pin_3), RV6.3
Other:
- note added: "MOD1"
- note added: "MOD1_LVL"
- note added: "MOD2"
- note added: "MOD2_LVL"
- note removed: "MOD_LVL"
- note removed: "Use as a second\nModulation input"
- moved on the sheet: R22, RV3
