File: KiCAD/AnVCO/Saw2Sqr.sch (KiCad schematic (older format))
At the start: 15 parts, among them J12 PWM, U4 TL072, U5 TL072

Commit message: Before wiring
Parts:
- R43: footprint Resistor_THT:R_Axial_DIN0207_L6.3mm_D2.5mm_P7.62mm_Horizontal -> Resistor_THT:R_Axial_DIN0207_L6.3mm_D2.5mm_P10.16mm_Horizontal
- renumbered J12 to J11, RV9 to RV10, RV8 to RV9, U5 to U4, U4 to U5
Connections:
- net SQR_OUT: now also U5.1, U5.2 (-); no longer U5.6 (-), U5.7
- net at RV10.2: now also U4.5 (+); no longer U4.3 (+)
- net at R38.1, R41.1: now also U5.3 (+); no longer U5.5 (+)
- new net: RV9.1, U4.6 (-), U4.7
Other:
- moved on the sheet: C17, C18
Changed lines of the file:
@@
 Sheet 5 5
 Title "AnVCO_Saw2Sqr"
-Date "2021-12-28"
+Date "2022-01-26"
 Rev "Ver. 1.0"
 Comp "PNPN Manufactory"
@@
 $Comp
 L Amplifier_Operational:TL072 U4
-U 1 1 606EF639
+U 2 1 606EF639
 P 4250 4050
 F 0 "U4" H 3950 4450 50  0000 C CNN
@@
 F 2 "Package_DIP:DIP-8_W7.62mm_Socket" H 4250 4050 50  0001 C CNN
 F 3 "http://www.ti.com/lit/ds/symlink/tl071.pdf" H 4250 4050 50  0001 C CNN
-	1    4250 4050
-	1    0    0    -1
-$EndComp
-$Comp
-L Amplifier_Operational:TL072 U4
+	2    4250 4050
+	1    0    0    -1
+$EndComp
+$Comp
+L Amplifier_Operational:TL072 U5
 U 2 1 606F0F43
 P 6100 3350
-F 0 "U4" H 6100 3717 50  0000 C CNN
+F 0 "U5" H 6100 3717 50  0000 C CNN
 F 1 "TL072" H 6100 3626 50  0000 C CNN
 F 2 "Package_DIP:DIP-8_W7.62mm_Socket" H 6100 3350 50  0001 C CNN
@@
 	3850 4700 4650 4700
 $Comp
-L Device:R_POT RV9
+L Device:R_POT RV10
 U 1 1 606FA9C6
 P 3600 3950
-F 0 "RV9" H 3530 3996 50  0000 R CNN
+F 0 "RV10" H 3530 3996 50  0000 R CNN
 F 1 "50kB" H 3530 3905 50  0000 R CNN
 F 2 "Potentiometer_THT:Potentiometer_Alps_RK097_Single_Horizontal" H 3600 3950 50  0001 C CNN
@@
 	3600 3400 3600 3350
 $Comp
-L Device:R_POT RV8
+L Device:R_POT RV9
 U 1 1 60700B29
 P 5050 3450
-F 0 "RV8" H 4981 3496 50  0000 R CNN
+F 0 "RV9" H 4981 3496 50  0000 R CNN
 F 1 "50kA" H 4981 3405 50  0000 R CNN
 F 2 "Potentiometer_THT:Potentiometer_Alps_RK097_Single_Horizontal" H 5050 3450 50  0001 C CNN
@@
 Connection ~ 4650 4050
 $Comp
-L Connector_Generic:Conn_01x02 J12
+L Connector_Generic:Conn_01x02 J11
 U 1 1 60701CE6
 P 3600 2800
-F 0 "J12" H 3518 3017 50  0000 C CNN
+F 0 "J11" H 3518 3017 50  0000 C CNN
 F 1 "PWM" H 3518 2926 50  0000 C CNN
 F 2 "Connector_JST:JST_XH_B2B-XH-A_1x02_P2.50mm_Vertical" H 3600 2800 50  0001 C CNN
@@
 $EndComp
 $Comp
-L power:-12V #PWR058
+L power:-12V #PWR059
 U 1 1 61CAC8A4
 P 4150 4450
-F 0 "#PWR058" H 4150 4550 50  0001 C CNN
+F 0 "#PWR059" H 4150 4550 50  0001 C CNN
 F 1 "-12V" H 4165 4623 50  0000 C CNN
 F 2 "" H 4150 4450 50  0001 C CNN
@@
 F 0 "R43" H 3670 4396 50  0000 L CNN
 F 1 "68k" H 3670 4305 50  0000 L CNN
-F 2 "Resistor_THT:R_Axial_DIN0207_L6.3mm_D2.5mm_P7.62mm_Horizontal" V 3530 4350 50  0001 C CNN
+F 2 "Resistor_THT:R_Axial_DIN0207_L6.3mm_D2.5mm_P10.16mm_Horizontal" V 3530 4350 50  0001 C CNN
 F 3 "~" H 3600 4350 50  0001 C CNN
 	1    3600 4350
@@
 $EndComp
 $Comp
-L power:-12V #PWR059
+L power:-12V #PWR061
 U 1 1 61CAD338
 P 3600 4550
-F 0 "#PWR059" H 3600 4650 50  0001 C CNN
+F 0 "#PWR061" H 3600 4650 50  0001 C CNN
 F 1 "-12V" H 3615 4723 50  0000 C CNN
 F 2 "" H 3600 4550 50  0001 C CNN
@@
 $Comp
 L Amplifier_Operational:TL072 U5
-U 2 1 61D069D2
+U 1 1 61D069D2
 P 7500 3450
-F 0 "U5" H 7500 3817 50  0000 C CNN
-F 1 "TL072" H 7500 3726 50  0000 C CNN
+F 0 "U5" H 7150 3850 50  0000 C CNN
+F 1 "TL072" H 7200 3750 50  0000 C CNN
 F 2 "Package_DIP:DIP-8_W7.62mm_Socket" H 7500 3450 50  0001 C CNN
 F 3 "http://www.ti.com/lit/ds/symlink/tl071.pdf" H 7500 3450 50  0001 C CNN
-	2    7500 3450
+	1    7500 3450
 	1    0    0    -1
 $EndComp
@@
 	7200 3550 7150 3550
 Wire Wire Line
-	7150 3550 7150 3850
-Wire Wire Line
-	7150 3850 7850 3850
-Wire Wire Line
-	7850 3850 7850 3450
+	7150 3550 7150 4100
+Wire Wire Line
+	7150 4100 7850 4100
+Wire Wire Line
+	7850 4100 7850 3450
 Wire Wire Line
 	7850 3450 7800 3450
@@
 Connection ~ 7850 3450
 $Comp
-L Amplifier_Operational:TL072 U5
+L Amplifier_Operational:TL072 U4
 U 1 1 61E4B5E3
 P 7500 4800
-F 0 "U5" H 7100 5150 50  0000 C CNN
+F 0 "U4" H 7100 5150 50  0000 C CNN
 F 1 "TL072" H 7150 5050 50  0000 C CNN
 F 2 "Package_DIP:DIP-8_W7.62mm_Socket" H 7500 4800 50  0001 C CNN
@@
 	7200 4900 7100 4900
 Wire Wire Line
-	7100 4900 7100 5450
-Wire Wire Line
-	7100 5450 7900 5450
-Wire Wire Line
-	7900 5450 7900 4800
+	7100 4900 7100 5150
+Wire Wire Line
+	7100 5150 7900 5150
+Wire Wire Line
+	7900 5150 7900 4800
 Wire Wire Line
 	7900 4800 7800 4800
@@
 L Amplifier_Operational:TL072 U5
 U 3 1 61E50407
-P 7500 4800
-F 0 "U5" H 7458 4846 50  0001 L CNN
-F 1 "TL072" H 7458 4755 50  0001 L CNN
-F 2 "Package_DIP:DIP-8_W7.62mm_Socket" H 7500 4800 50  0001 C CNN
-F 3 "http://www.ti.com/lit/ds/symlink/tl071.pdf" H 7500 4800 50  0001 C CNN
-	3    7500 4800
+P 7500 3450
+F 0 "U5" H 7458 3496 50  0001 L CNN
+F 1 "TL072" H 7458 3405 50  0001 L CNN
+F 2 "Package_DIP:DIP-8_W7.62mm_Socket" H 7500 3450 50  0001 C CNN
+F 3 "http://www.ti.com/lit/ds/symlink/tl071.pdf" H 7500 3450 50  0001 C CNN
+	3    7500 3450
 	1    0    0    -1
 $EndComp
@@
 L Device:C C17
 U 1 1 61E5942E
-P 7550 4450
-F 0 "C17" V 7300 4500 50  0000 C CNN
-F 1 "0.1uF" V 7400 4500 50  0000 C CNN
-F 2 "Capacitor_THT:C_Disc_D3.0mm_W1.6mm_P2.50mm" H 7588 4300 50  0001 C CNN
-F 3 "~" H 7550 4450 50  0001 C CNN
-	1    7550 4450
+P 7550 3100
+F 0 "C17" V 7300 3150 50  0000 C CNN
+F 1 "0.1uF" V 7400 3150 50  0000 C CNN
+F 2 "Capacitor_THT:C_Disc_D3.0mm_W1.6mm_P2.50mm" H 7588 2950 50  0001 C CNN
+F 3 "~" H 7550 3100 50  0001 C CNN
+	1    7550 3100
 	0    1    1    0
 $EndComp
 $Comp
-L power:GND #PWR061
+L power:GND #PWR060
 U 1 1 61E59434
-P 7700 4450
-F 0 "#PWR061" H 7700 4200 50  0001 C CNN
-F 1 "GND" V 7705 4322 50  0000 R CNN
-F 2 "" H 7700 4450 50  0001 C CNN
-F 3 "" H 7700 4450 50  0001 C CNN
-	1    7700 4450
-	0    -1   -1   0
-$EndComp
-Wire Wire Line
-	7400 4400 7400 4450
-Wire Wire Line
-	7400 4500 7400 4450
-Connection ~ 7400 4450
-$Comp
-L power:+12V #PWR060
+P 7700 3100
+F 0 "#PWR060" H 7700 2850 50  0001 C CNN
+F 1 "GND" V 7705 2972 50  0000 R CNN
+F 2 "" H 7700 3100 50  0001 C CNN
+F 3 "" H 7700 3100 50  0001 C CNN
+	1    7700 3100
+	0    -1   -1   0
+$EndComp
+Wire Wire Line
+	7400 3050 7400 3100
+Wire Wire Line
+	7400 3150 7400 3100
+Connection ~ 7400 3100
+$Comp
+L power:+12V #PWR058
 U 1 1 61E5943D
-P 7400 4400
-F 0 "#PWR060" H 7400 4250 50  0001 C CNN
-F 1 "+12V" H 7415 4573 50  0000 C CNN
-F 2 "" H 7400 4400 50  0001 C CNN
-F 3 "" H 7400 4400 50  0001 C CNN
-	1    7400 4400
+P 7400 3050
+F 0 "#PWR058" H 7400 2900 50  0001 C CNN
+F 1 "+12V" H 7415 3223 50  0000 C CNN
+F 2 "" H 7400 3050 50  0001 C CNN
+F 3 "" H 7400 3050 50  0001 C CNN
+	1    7400 3050
 	1    0    0    -1
 $EndComp
@@
 L Device:C C18
 U 1 1 61E5B63E
-P 7550 5150
-F 0 "C18" V 7800 5050 50  0000 C CNN
-F 1 "0.1uF" V 7700 5050 50  0000 C CNN
-F 2 "Capacitor_THT:C_Disc_D3.0mm_W1.6mm_P2.50mm" H 7588 5000 50  0001 C CNN
-F 3 "~" H 7550 5150 50  0001 C CNN
-	1    7550 5150
+P 7550 3800
+F 0 "C18" V 7800 3700 50  0000 C CNN
+F 1 "0.1uF" V 7700 3700 50  0000 C CNN
+F 2 "Capacitor_THT:C_Disc_D3.0mm_W1.6mm_P2.50mm" H 7588 3650 50  0001 C CNN
+F 3 "~" H 7550 3800 50  0001 C CNN
+	1    7550 3800
 	0    -1   -1   0
 $EndComp
@@
 L power:GND #PWR063
 U 1 1 61E5B648
-P 7700 5150
-F 0 "#PWR063" H 7700 4900 50  0001 C CNN
-F 1 "GND" V 7705 5022 50  0000 R CNN
-F 2 "" H 7700 5150 50  0001 C CNN
-F 3 "" H 7700 5150 50  0001 C CNN
-	1    7700 5150
-	0    -1   -1   0
-$EndComp
-Wire Wire Line
-	7400 5100 7400 5150
-Wire Wire Line
-	7400 5200 7400 5150
-Connection ~ 7400 5150
+P 7700 3800
+F 0 "#PWR063" H 7700 3550 50  0001 C CNN
+F 1 "GND" V 7705 3672 50  0000 R CNN
+F 2 "" H 7700 3800 50  0001 C CNN
+F 3 "" H 7700 3800 50  0001 C CNN
+	1    7700 3800
+	0    -1   -1   0
+$EndComp
+Wire Wire Line
+	7400 3750 7400 3800
+Wire Wire Line
+	7400 3850 7400 3800
+Connection ~ 7400 3800
 $Comp
 L power:-12V #PWR064
 U 1 1 61E5B655
-P 7400 5200
-F 0 "#PWR064" H 7400 5300 50  0001 C CNN
-F 1 "-12V" H 7415 5373 50  0000 C CNN
-F 2 "" H 7400 5200 50  0001 C CNN
-F 3 "" H 7400 5200 50  0001 C CNN
-	1    7400 5200
+P 7400 3850
+F 0 "#PWR064" H 7400 3950 50  0001 C CNN
+F 1 "-12V" H 7415 4023 50  0000 C CNN
+F 2 "" H 7400 3850 50  0001 C CNN
+F 3 "" H 7400 3850 50  0001 C CNN
+	1    7400 3850
 	-1   0    0    1
 $EndComp
