File: KiCAD/AnVCO/Saw2Tri.sch (KiCad schematic (older format))
At the start: 11 parts, among them Q4 2SC1815, U3 TL072

Commit message: Before wiring
Parts:
- RV8: renamed from RV7; footprint Connector_JST:JST_XH_B3B-XH-A_1x03_P2.50mm_Vertical -> Potentiometer_THT:Potentiometer_Bourns_3296W_Vertical
Changed lines of the file:
@@
 Sheet 4 5
 Title "AnVCO_Saw2Tri"
-Date "2021-12-28"
+Date "2022-01-26"
 Rev "Ver. 1.0"
 Comp "PNPN Manufactory"
@@
 $EndComp
 $Comp
-L Device:R_POT_TRIM RV7
+L Device:R_POT_TRIM RV8
 U 1 1 603FFFCF
 P 5400 3150
-F 0 "RV7" H 5330 3104 50  0000 R CNN
+F 0 "RV8" H 5330 3104 50  0000 R CNN
 F 1 "5k" H 5330 3195 50  0000 R CNN
-F 2 "Connector_JST:JST_XH_B3B-XH-A_1x03_P2.50mm_Vertical" H 5400 3150 50  0001 C CNN
+F 2 "Potentiometer_THT:Potentiometer_Bourns_3296W_Vertical" H 5400 3150 50  0001 C CNN
 F 3 "~" H 5400 3150 50  0001 C CNN
 	1    5400 3150
