File: KiCAD/AnVCO/SawVCO.sch (KiCad schematic (older format))
At the start: 20 parts, among them J10 Sync_In, J11 Liner_FM, Q3 2SA1015, U2 TL072

Commit message: Before wiring
Parts:
- removed J10: Sync_In, Connector_JST:JST_XH_B2B-XH-A_1x02_P2.50mm_Vertical, symbol Connector_Generic:Conn_01x02
- removed J11: Liner_FM, Connector_JST:JST_XH_B2B-XH-A_1x02_P2.50mm_Vertical, symbol Connector_Generic:Conn_01x02
- added J10: Sync&FM, Connector_JST:JST_XH_B4B-XH-A_1x04_P2.50mm_Vertical, symbol Connector_Generic:Conn_01x04
- RV7: renamed from RV6; footprint Potentiometer_THT:Potentiometer_Bourns_3296X_Horizontal -> Potentiometer_THT:Potentiometer_Bourns_3296W_Vertical
Connections:
- net GND: now also J10.2 (Pin_2), J10.4 (Pin_4)
- net I_SINK: now also U2.5 (+); no longer U2.3 (+)
- net SAW_OUT: now also U2.7; no longer U2.1
- net at C7.2, R26.1: now also U2.1; no longer U2.7
- net at R29.1, R32.1: now also U2.6 (-); no longer U2.2 (-)
- net at C10.2: now also J10.3 (Pin_3)
- net at C7.1, R24.2, R28.1: now also R23.1, U2.3 (+); no longer R23.2, U2.5 (+)
- net at R30.1: now also U2.2 (-); no longer U2.6 (-)
- new net: J10.1 (Pin_1), R23.2
Other:
- note added: "LinerFM"
- note added: "SyncIn"
- moved on the sheet: C10, C11, C7, C8, C9, Q3, R23, R24, R25, R26, R27, R28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
