File: KiCAD/AnVCO/AnVCO.kicad_pcb (KiCad board)
At the start: 2 copper layers, 99.7 x 99.7 mm, 103 parts, among them J1 CV, J10 Sync&FM, J11 PWM, J2 SW_WaveForm, J3 OUT, J4 ERK_PWR, J5 TP_GND, J6 TP_GND, J7 MSTR_OUT, J8 COURSE_SW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

Commit message: Ver.1.0
Parts:
- added G***: LOGO, myfootprint:Silk_PNPN_Thyristor_1200dpi, F.Cu at (147.3, 116.8)
- added G***: LOGO, myfootprint:Silk_PNPN_Manufactory_600dpi, F.Cu at (137.2, 114.3)
- moved TP1 32.6 mm to (135.9, 78.7)
- moved R24 10.2 mm to (130.8, 95.2), turned to 0 degrees
Routing:
- net -12V: track 0.00 -> 322.5 mm
- net +12V: track 0.00 -> 275.4 mm
- net +5V: track 0.00 -> 185.6 mm, vias 0 -> 2
- net /Antilog_NPNO/CV: track 0.00 -> 158.3 mm
- net /Saw2Sqr/SAW_IN: track 0.00 -> 106.8 mm, vias 0 -> 2
- net Net-(R10-Pad2): track 0.00 -> 103.1 mm
- net /Saw2Sqr/SQR_OUT: track 0.00 -> 77.4 mm
- net /Antilog_NPNO/VREF: track 0.00 -> 68.2 mm
- net Net-(J10-Pad1): track 0.00 -> 58.5 mm
- net /Antilog_NPNO/I_SINK: track 0.00 -> 55.6 mm
- net Net-(C7-Pad1): track 0.00 -> 46.5 mm
- net Net-(J11-Pad1): track 0.00 -> 45.5 mm
- net /Saw2Tri/TRI_OUT: track 0.00 -> 43.0 mm
- net Net-(C10-Pad2): track 0.00 -> 37.8 mm
- net Net-(R20-Pad1): track 0.00 -> 37.4 mm
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- added copper zone on F.Cu, net GND
Other:
- board text added: "+12V"
- board text added: "AnVCO"
- board text added: "COM G COURSE_SW"
- board text added: "COM SAW TRI SQR"
- board text added: "COURCE_ADJ"
- board text added: "CV"
- board text added: "CV_ADJ"
- board text added: "CV_COM"
- board text added: "FINE"
- board text added: "G CV"
- board text added: "G MOD2 G MOD1"
- board text added: "G MSTR_OUT"
- board text added: "G PWM"
- board text added: "G SQR G OUT"
- board text added: "GND"
- board text added: "HIGH_ADJ"
- board text added: "I_SINK"
- board text added: "MOD1"
- board text added: "MOD2"
- board text added: "OUT"
- board text added: "PW"
- board text added: "PWM"
- board text added: "SCALE"
- board text added: "SYNC G FM G"
- board text added: "TRI_SHAPE"
- board text added: "VREF"
- board text added: "Ver. 1.0"
- board text added: "WAVE_FORM_SW"
- board text added: "https://dad8893.blogspot.com/"
